File: Week_2/Week_2_Activity/Audio_Board/Audio_Board.sch (KiCad schematic (older format))
At the start: 105 parts, among them J1 1017523, J2 801-47-018-10-012000, J3 310-87-114-41-001101, J4 PBC03SAAN, J5 1017523, J6 1017521, J7 1017521, U1 VS1053B, U10 MOUNTINGHOLE2.5_THICK, U11 MOUNTINGHOLE2.5_THICK, U12 MOUNTINGHOLE2.5_THICK, U2 AP7312-1833W6-7, U3 MAX1735EUK25-T, U4 ADA4807-2, U5 ADA4807-2, U6 TC1262-2.5VDB, U7 MC78M12ABDTRKG, U8 TPA3250D2DDW, U9 MOUNTINGHOLE2.5_THICK, Y1 ABM8G-

Commit message: Update Audio_Board.sch
Parts:
- C29: value 0.1µF -> 0.01µF
Changed lines of the file:
@@
 P 9350 7050
 F 0 "C29" H 9465 7096 50  0000 L CNN
-F 1 "0.1µF" H 9465 7005 50  0000 L CNN
+F 1 "0.01µF" H 9465 7005 50  0000 L CNN
 F 2 "" H 9388 6900 50  0001 C CNN
 F 3 "~" H 9350 7050 50  0001 C CNN
