File: Overview & Details/Week_3/Week_3_Activity/Activity_3/activity3/TFT_LCD.sch (KiCad schematic (older format))
At the start: 37 parts, among them IC1 MIC5225-3.3, IC2 74LVC245, IC3 74LVC245, IC4 APX803-SAG, Q1 MMBT2222, X1 MICROSD

Commit message: made connections local to the STMPE811. removed TFT_LCD schematic. annotated schematic
Parts:
- removed C1, C4: 0.1uF, Adafruit 2.8 TFT Breakout v2:0805-NO, symbol Adafruit_2.8_TFT_Breakout_v2-eagle-import:CAP_CERAMIC0805-NOOUTLINE
- removed C2, C3, C5: 10uF, Adafruit 2.8 TFT Breakout v2:0805-NO, symbol Adafruit_2.8_TFT_Breakout_v2-eagle-import:CAP_CERAMIC0805-NOOUTLINE
- removed IC1: MIC5225-3.3, Adafruit 2.8 TFT Breakout v2:SOT23-5L, symbol Adafruit_2.8_TFT_Breakout_v2-eagle-import:LP298XS
- removed IC2, IC3: 74LVC245, Adafruit 2.8 TFT Breakout v2:SO20W, symbol Adafruit_2.8_TFT_Breakout_v2-eagle-import:74245DW
- removed IC4: APX803-SAG, Adafruit 2.8 TFT Breakout v2:SOT23, symbol Adafruit_2.8_TFT_Breakout_v2-eagle-import:AXP083-SAG
- removed JP1, JP2: HEADER-1X20ROUND, Adafruit 2.8 TFT Breakout v2:1X20_ROUND, symbol Adafruit_2.8_TFT_Breakout_v2-eagle-import:HEADER-1X20ROUND
- removed Q1: MMBT2222, Adafruit 2.8 TFT Breakout v2:SOT23-BEC, symbol Adafruit_2.8_TFT_Breakout_v2-eagle-import:-NPN-SOT23-BEC
- removed R1, R2, R3, R4: 10, Adafruit 2.8 TFT Breakout v2:0805-NO, symbol Adafruit_2.8_TFT_Breakout_v2-eagle-import:RESISTOR0805_NOOUTLINE
- removed R10, R11, R12, R8, R9: 10K, Adafruit 2.8 TFT Breakout v2:0805-NO, symbol Adafruit_2.8_TFT_Breakout_v2-eagle-import:RESISTOR0805_NOOUTLINE
- removed R5, R7: 1K, Adafruit 2.8 TFT Breakout v2:0805-NO, symbol Adafruit_2.8_TFT_Breakout_v2-eagle-import:RESISTOR0805_NOOUTLINE
- removed R6: 10K, Adafruit 2.8 TFT Breakout v2:R0805, symbol Adafruit_2.8_TFT_Breakout_v2-eagle-import:R-US_R0805
- removed SJ1, SJ2, SJ3, SJ4: SOLDERJUMPER, Adafruit 2.8 TFT Breakout v2:SOLDERJUMPER_ARROW_NOPASTE, symbol Adafruit_2.8_TFT_Breakout_v2-eagle-import:SOLDERJUMPER
- removed U$10: DISP_LCD_1.28IN_240X320_50PIN, Adafruit 2.8 TFT Breakout v2:TFT_2.83IN_240X320_50PIN, symbol Adafruit_2.8_TFT_Breakout_v2-eagle-import:DISP_LCD_1.28IN_240X320_50PIN
- removed U$11, U$23, U$9: FIDUCIAL, Adafruit 2.8 TFT Breakout v2:FIDUCIAL_1MM, symbol Adafruit_2.8_TFT_Breakout_v2-eagle-import:FIDUCIAL
- removed U$15, U$16, U$17, U$7: MOUNTINGHOLE3.0THIN, Adafruit 2.8 TFT Breakout v2:MOUNTINGHOLE_3.0_PLATEDTHIN, symbol Adafruit_2.8_TFT_Breakout_v2-eagle-import:MOUNTINGHOLE3.0THIN
- removed X1: MICROSD, Adafruit 2.8 TFT Breakout v2:MICROSD, symbol Adafruit_2.8_TFT_Breakout_v2-eagle-import:MICROSD
Connections:
- net labels removed: +5V, CARDDET, FRAME_A4_ADAFRUIT, GND, IM0, IM1, IM2, IM3, LCD_CS, LCD_CS_5V, LCD_DATA0, LCD_DATA0_5V, LCD_DATA1, LCD_DATA1_5V, LCD_DATA2, LCD_DATA2_5V, LCD_DATA3, LCD_DATA3_5V, LCD_DATA4, LCD_DATA4_5V, LCD_DATA5, LCD_DATA5_5V, LCD_DATA6, LCD_DATA6_5V, LCD_DATA7, LCD_DATA7_5V, LCD_LITE, LCD_RD, LCD_RD_5V, LCD_RS, LCD_RST, LCD_RST_5V, LCD_RS_5V, LCD_WR, LCD_WR_5V, LCD_X+, LCD_X-, LCD_Y+, LCD_Y-, SDI_3V, SDI_5V, SDO, SD_CS_3V, SD_CS_5V, VCC
- wire segments 162 -> 0
