File: Overview & Details/Audioboard/Audioboard_Activity/Audio_Board/Audio_Board.sch (KiCad schematic (older format))
At the start: 105 parts, among them J1 1017523, J2 801-47-018-10-012000, J3 310-87-114-41-001101, J4 PBC03SAAN, J5 1017523, J6 1017521, J7 1017521, U1 VS1053B, U10 MOUNTINGHOLE2.5_THICK, U11 MOUNTINGHOLE2.5_THICK, U12 MOUNTINGHOLE2.5_THICK, U2 AP7312-1833W6-7, U3 MAX1735EUK25-T, U4 ADA4807-2, U5 ADA4807-2, U6 TC1262-2.5VDB, U7 MC78M12ABDTRKG, U8 TPA3250D2DDW, U9 MOUNTINGHOLE2.5_THICK, Y1 ABM8G-

Commit message: Added footprints to audioboard
Parts:
- C1, C12, C13, C14, C15, C16, C18, C19, C2, C20, C21, C22, C23, C24, C25, C26, C29, C3, C32, C33, C36, C37, C38, C39, C4, C40, C41, C42, C43, C44, C45, C46, C47, C48, C49, C5, C58, C59, C6, C60, C61, C7, C8, C9: footprint (none) -> Capacitor_SMD:C_0603_1608Metric
- C10, C11: footprint (none) -> Capacitor_SMD:CP_Elec_8x11.9
- C27, C28: footprint (none) -> Capacitor_THT:C_Radial_D18.0mm_H35.5mm_P7.50mm
- C30, C31, C34, C35, C54, C55, C56, C57: footprint (none) -> Capacitor_SMD:C_1206_3216Metric
- C50, C51: footprint (none) -> Capacitor_THT:C_Radial_D16.0mm_H31.5mm_P7.50mm
- C52, C53: footprint (none) -> Capacitor_THT:C_Radial_D16.0mm_H25.0mm_P7.50mm
- FB1, FB2: footprint (none) -> Inductor_SMD:L_0603_1608Metric; symbol Adafruit_VS1053_Breakout-eagle-import:FERRITE_0603 -> Audio_Board-rescue:FERRITE_0603-Adafruit_VS1053_Breakout-eagle-import
- J1, J5: footprint (none) -> TerminalBlock_Phoenix:PhoenixContact_TermBlk_4P_SideEnt_6.35MM
- J4: footprint (none) -> Connector_PinHeader_2.54mm:PinHeader_1x03_P2.54mm_Vertical
- J6, J7: footprint (none) -> TerminalBlock_Phoenix:PhoenixContact_TermBlk_2P_SideEnt_6.35MM
- L1, L2, L3, L4: footprint (none) -> Inductor_THT:L_Toroid_Vertical_L26.7mm_W14.0mm_P10.16mm_Pulse_D
- R1, R10, R13, R14, R15, R16, R17, R18, R3, R4, R5, R6, R9: footprint (none) -> Resistor_SMD:R_0603_1608Metric
- R2: footprint (none) -> Resistor_SMD:R_0805_2012Metric
- U1: footprint (none) -> Package_QFP:LQFP-48_7x7mm_P0.5mm; symbol Adafruit_VS1053_Breakout-eagle-import:VS1053B -> Audio_Board-rescue:VS1053B-Adafruit_VS1053_Breakout-eagle-import
- U10, U11, U12, U9: symbol Adafruit_VS1053_Breakout-eagle-import:MOUNTINGHOLE2.5_THICK -> Audio_Board-rescue:MOUNTINGHOLE2.5_THICK-Adafruit_VS1053_Breakout-eagle-import
- U2: footprint (none) -> Package_TO_SOT_SMD:SOT-23-6; symbol Adafruit_VS1053_Breakout-cache:Adafruit_VS1053_Breakout-eagle-import_VREG_SOT23-6_DUALAP7312 -> Audio_Board-rescue:Adafruit_VS1053_Breakout-eagle-import_VREG_SOT23-6_DUALAP7312-Adafruit_VS1053_Breakout-cache
- U4, U5: footprint (none) -> Package_SO:MSOP-8_3x3mm_P0.65mm
- U6: footprint (none) -> Package_TO_SOT_SMD:SOT-223-3_TabPin2
- Y1: footprint (none) -> Crystal:Crystal_SMD_Abracon_ABM8G-4Pin_3.2x2.5mm; symbol Adafruit_VS1053_Breakout-eagle-import:CRYSTAL3.2X2.5 -> Audio_Board-rescue:CRYSTAL3.2X2.5-Adafruit_VS1053_Breakout-eagle-import

Commit message: created footprint for circular pins for sam32 and linked to symbols. linked displayboard's lcd screen to the 50pin connector footprint
Parts:
- C17: footprint (none) -> Capacitor_SMD:C_0603_1608Metric
- J2: footprint (none) -> Audio_Board:801-47-018-10-012000
- J3: footprint (none) -> Audio_Board:310-87-114-41-001101
Changed lines of the file:
@@
 F 0 "C17" V 7650 5100 50  0000 C CNN
 F 1 "22pF" V 7650 5400 50  0000 C CNN
-F 2 "" H 7550 5200 50  0001 C CNN
+F 2 "Capacitor_SMD:C_0603_1608Metric" H 7550 5200 50  0001 C CNN
 F 3 "~" H 7550 5200 50  0001 C CNN
 	1    7550 5200
@@
 F 0 "J3" H 4192 9685 50  0000 C CNN
 F 1 "310-87-114-41-001101 " H 4000 8000 50  0000 C CNN
-F 2 "" H 4300 8900 50  0001 C CNN
+F 2 "Audio_Board:310-87-114-41-001101" H 4300 8900 50  0001 C CNN
 F 3 "~" H 4300 8900 50  0001 C CNN
 	1    4300 8900
@@
 F 0 "J2" H 2600 9800 50  0000 L CNN
 F 1 "801-47-018-10-012000" H 2000 7800 50  0000 L CNN
-F 2 "" H 2800 8800 50  0001 C CNN
+F 2 "Audio_Board:801-47-018-10-012000" H 2800 8800 50  0001 C CNN
 F 3 "~" H 2800 8800 50  0001 C CNN
 	1    2800 8800

Commit message: finished assigning audioboard footprints
Parts:
- C54, C55, C56, C57: footprint Capacitor_SMD:C_1206_3216Metric -> Audio_Board:ADA4807-2ACPZ-R2
- R11, R12, R7, R8: footprint (none) -> Resistor_SMD:R_0603_1608Metric
- U10, U11, U12, U9: footprint (none) -> MountingHole:MountingHole_2.5mm
- U4, U5: footprint Package_SO:MSOP-8_3x3mm_P0.65mm -> Audio_Board:ADA4807-2ACPZ-R2
- U4, U5: footprint (none) -> Audio_Board:ADA4807-2ACPZ-R2
- U8: footprint DDW0044A_N -> Audio_Board:TPA3250D2DDWR
Changed lines of the file:
@@
 F 0 "C54" H 14765 2796 50  0000 L CNN
 F 1 "1nF" H 14765 2705 50  0000 L CNN
-F 2 "Capacitor_SMD:C_1206_3216Metric" H 14688 2600 50  0001 C CNN
+F 2 "Audio_Board:ADA4807-2ACPZ-R2" H 14688 2600 50  0001 C CNN
 F 3 "https://search.murata.co.jp/Ceramy/image/img/A01X/G101/ENG/GRM3195C1H102JA01-01.pdf" H 14650 2750 50  0001 C CNN
 F 4 "Capacitor, Ceramic, 1000pF, 50V, 5%, C0G/NP0, 1206" H 14650 2750 50  0001 C CNN "Description"
@@
 F 0 "U4" H 7450 4100 50  0000 C CNN
 F 1 "ADA4807-2" H 7550 3850 50  0000 C CNN
-F 2 "Package_SO:MSOP-8_3x3mm_P0.65mm" H 7500 4100 50  0001 C CNN
+F 2 "Audio_Board:ADA4807-2ACPZ-R2" H 7500 4100 50  0001 C CNN
 F 3 "http://www.analog.com/media/en/technical-documentation/data-sheets/ADA4807-1_4807-2_4807-4.pdf" H 7500 4100 50  0001 C CNN
 F 4 "IC, 3.1 nV/√Hz, 1 mA, 180 MHz, Rail-to-Rail Input/Output Amplifier, Dual" H 7500 4100 50  0001 C CNN "Description"
@@
 F 0 "U4" H 7450 4700 50  0000 C CNN
 F 1 "ADA4807-2" H 7550 4450 50  0000 C CNN
-F 2 "" H 7500 4700 50  0001 C CNN
+F 2 "Audio_Board:ADA4807-2ACPZ-R2" H 7500 4700 50  0001 C CNN
 F 3 "http://www.analog.com/media/en/technical-documentation/data-sheets/ADA4807-1_4807-2_4807-4.pdf" H 7500 4700 50  0001 C CNN
 F 4 "IC, 3.1 nV/√Hz, 1 mA, 180 MHz, Rail-to-Rail Input/Output Amplifier, Dual" H 7500 4700 50  0001 C CNN "Description"
@@
 F 0 "U4" V 7450 3400 50  0000 L CNN
 F 1 "ADA4807-2" V 7250 3200 50  0000 L CNN
-F 2 "" H 7450 3500 50  0001 C CNN
+F 2 "Audio_Board:ADA4807-2ACPZ-R2" H 7450 3500 50  0001 C CNN
 F 3 "http://www.analog.com/media/en/technical-documentation/data-sheets/ADA4807-1_4807-2_4807-4.pdf" H 7450 3500 50  0001 C CNN
 F 4 "IC, 3.1 nV/√Hz, 1 mA, 180 MHz, Rail-to-Rail Input/Output Amplifier, Dual" V 7450 3500 50  0001 C CNN "Description"
@@
 F 0 "R8" V 7150 4500 50  0000 L CNN
 F 1 "10.0k" V 7150 4700 50  0000 L CNN
-F 2 "" V 7090 4790 50  0001 C CNN
+F 2 "Resistor_SMD:R_0603_1608Metric" V 7090 4790 50  0001 C CNN
 F 3 "~" H 7050 4800 50  0001 C CNN
 	1    7050 4800
@@
 F 0 "R12" V 7600 4800 50  0000 L CNN
 F 1 "10.0k" V 7600 5150 50  0000 L CNN
-F 2 "" V 7590 5040 50  0001 C CNN
+F 2 "Resistor_SMD:R_0603_1608Metric" V 7590 5040 50  0001 C CNN
 F 3 "~" H 7550 5050 50  0001 C CNN
 	1    7550 5050
@@
 F 0 "U5" H 7450 5600 50  0000 C CNN
 F 1 "ADA4807-2" H 7550 5350 50  0000 C CNN
-F 2 "Package_SO:MSOP-8_3x3mm_P0.65mm" H 7500 5600 50  0001 C CNN
+F 2 "Audio_Board:ADA4807-2ACPZ-R2" H 7500 5600 50  0001 C CNN
 F 3 "http://www.analog.com/media/en/technical-documentation/data-sheets/ADA4807-1_4807-2_4807-4.pdf" H 7500 5600 50  0001 C CNN
 F 4 "IC, 3.1 nV/√Hz, 1 mA, 180 MHz, Rail-to-Rail Input/Output Amplifier, Dual" H 7500 5600 50  0001 C CNN "Description"
@@
 F 0 "U5" H 7450 6200 50  0000 C CNN
 F 1 "ADA4807-2" H 7550 5950 50  0000 C CNN
-F 2 "" H 7500 6200 50  0001 C CNN
+F 2 "Audio_Board:ADA4807-2ACPZ-R2" H 7500 6200 50  0001 C CNN
 F 3 "http://www.analog.com/media/en/technical-documentation/data-sheets/ADA4807-1_4807-2_4807-4.pdf" H 7500 6200 50  0001 C CNN
 F 4 "IC, 3.1 nV/√Hz, 1 mA, 180 MHz, Rail-to-Rail Input/Output Amplifier, Dual" H 7500 6200 50  0001 C CNN "Description"
@@
 F 0 "U5" V 7350 7000 50  0000 L CNN
 F 1 "ADA4807-2" V 7550 6800 50  0000 L CNN
-F 2 "" H 7550 7100 50  0001 C CNN
+F 2 "Audio_Board:ADA4807-2ACPZ-R2" H 7550 7100 50  0001 C CNN
 F 3 "http://www.analog.com/media/en/technical-documentation/data-sheets/ADA4807-1_4807-2_4807-4.pdf" H 7550 7100 50  0001 C CNN
 F 4 "IC, 3.1 nV/√Hz, 1 mA, 180 MHz, Rail-to-Rail Input/Output Amplifier, Dual" V 7550 7100 50  0001 C CNN "Description"
@@
 F 0 "R11" V 7550 6300 50  0000 L CNN
 F 1 "10.0k" V 7550 6650 50  0000 L CNN
-F 2 "" V 7540 6540 50  0001 C CNN
+F 2 "Resistor_SMD:R_0603_1608Metric" V 7540 6540 50  0001 C CNN
 F 3 "~" H 7500 6550 50  0001 C CNN
 	1    7500 6550
@@
 F 0 "U12" H 12100 10400 50  0001 C CNN
 F 1 "MOUNTINGHOLE2.5_THICK" H 12050 10350 50  0001 C CNN
-F 2 "" H 12050 10350 50  0001 C CNN
+F 2 "MountingHole:MountingHole_2.5mm" H 12050 10350 50  0001 C CNN
 F 3 "" H 12050 10350 50  0001 C CNN
 	1    12050 10350
@@
 F 0 "U11" H 12100 10150 50  0001 C CNN
 F 1 "MOUNTINGHOLE2.5_THICK" H 12050 10100 50  0001 C CNN
-F 2 "" H 12050 10100 50  0001 C CNN
+F 2 "MountingHole:MountingHole_2.5mm" H 12050 10100 50  0001 C CNN
 F 3 "" H 12050 10100 50  0001 C CNN
 	1    12050 10100
@@
 F 0 "U10" H 12100 9900 50  0001 C CNN
 F 1 "MOUNTINGHOLE2.5_THICK" H 12050 9850 50  0001 C CNN
-F 2 "" H 12050 9850 50  0001 C CNN
+F 2 "MountingHole:MountingHole_2.5mm" H 12050 9850 50  0001 C CNN
 F 3 "" H 12050 9850 50  0001 C CNN
 	1    12050 9850
@@
 F 0 "U9" H 12100 9650 50  0001 C CNN
 F 1 "MOUNTINGHOLE2.5_THICK" H 12050 9600 50  0001 C CNN
-F 2 "" H 12050 9600 50  0001 C CNN
+F 2 "MountingHole:MountingHole_2.5mm" H 12050 9600 50  0001 C CNN
 F 3 "" H 12050 9600 50  0001 C CNN
 	1    12050 9600
@@
 F 0 "R7" V 6950 4450 50  0000 L CNN
 F 1 "5.0k" V 6950 4600 50  0000 L CNN
-F 2 "" V 7090 4590 50  0001 C CNN
+F 2 "Resistor_SMD:R_0603_1608Metric" V 7090 4590 50  0001 C CNN
 F 3 "~" H 7050 4600 50  0001 C CNN
 	1    7050 4600
@@
 F 0 "U8" H 11350 7888 60  0000 C CNN
 F 1 "TPA3250D2DDW" H 11350 7782 60  0000 C CNN
-F 2 "DDW0044A_N" H 11350 5240 60  0001 C CNN
+F 2 "Audio_Board:TPA3250D2DDWR" H 11350 5240 60  0001 C CNN
 F 3 "https://www.ti.com/lit/ds/symlink/tpa3250.pdf" H 11350 5300 60  0001 C CNN
 F 4 "50-W Stereo, 175W peak Ultra-HD Pad Down Class-D Amplifier" H 11350 5300 50  0001 C CNN "Description"
@@
 F 0 "C55" H 14765 3896 50  0000 L CNN
 F 1 "1nF" H 14765 3805 50  0000 L CNN
-F 2 "Capacitor_SMD:C_1206_3216Metric" H 14688 3700 50  0001 C CNN
+F 2 "Audio_Board:ADA4807-2ACPZ-R2" H 14688 3700 50  0001 C CNN
 F 3 "https://search.murata.co.jp/Ceramy/image/img/A01X/G101/ENG/GRM3195C1H102JA01-01.pdf" H 14650 3850 50  0001 C CNN
 F 4 "Capacitor, Ceramic, 1000pF, 50V, 5%, C0G/NP0, 1206" H 14650 3850 50  0001 C CNN "Description"
@@
 F 0 "C56" H 14765 5096 50  0000 L CNN
 F 1 "1nF" H 14765 5005 50  0000 L CNN
-F 2 "Capacitor_SMD:C_1206_3216Metric" H 14688 4900 50  0001 C CNN
+F 2 "Audio_Board:ADA4807-2ACPZ-R2" H 14688 4900 50  0001 C CNN
 F 3 "https://search.murata.co.jp/Ceramy/image/img/A01X/G101/ENG/GRM3195C1H102JA01-01.pdf" H 14650 5050 50  0001 C CNN
 F 4 "Capacitor, Ceramic, 1000pF, 50V, 5%, C0G/NP0, 1206" H 14650 5050 50  0001 C CNN "Description"
@@
 F 0 "C57" H 14765 6146 50  0000 L CNN
 F 1 "1nF" H 14765 6055 50  0000 L CNN
-F 2 "Capacitor_SMD:C_1206_3216Metric" H 14688 5950 50  0001 C CNN
+F 2 "Audio_Board:ADA4807-2ACPZ-R2" H 14688 5950 50  0001 C CNN
 F 3 "https://search.murata.co.jp/Ceramy/image/img/A01X/G101/ENG/GRM3195C1H102JA01-01.pdf" H 14650 6100 50  0001 C CNN
 F 4 "Capacitor, Ceramic, 1000pF, 50V, 5%, C0G/NP0, 1206" H 14650 6100 50  0001 C CNN "Description"

Commit message: added footprints for square stackable pins (for sam32)
Parts:
- J2: footprint Audio_Board:801-47-018-10-012000 -> Audio_Board:SSQ-117-03-F-S
- J3: footprint Audio_Board:310-87-114-41-001101 -> Audio_Board:SSQ-114-03-F-S
Changed lines of the file:
@@
 F 0 "J3" H 4192 9685 50  0000 C CNN
 F 1 "310-87-114-41-001101 " H 4000 8000 50  0000 C CNN
-F 2 "Audio_Board:310-87-114-41-001101" H 4300 8900 50  0001 C CNN
+F 2 "Audio_Board:SSQ-114-03-F-S" H 4300 8900 50  0001 C CNN
 F 3 "~" H 4300 8900 50  0001 C CNN
 	1    4300 8900
@@
 F 0 "J2" H 2600 9800 50  0000 L CNN
 F 1 "801-47-018-10-012000" H 2000 7800 50  0000 L CNN
-F 2 "Audio_Board:801-47-018-10-012000" H 2800 8800 50  0001 C CNN
+F 2 "Audio_Board:SSQ-117-03-F-S" H 2800 8800 50  0001 C CNN
 F 3 "~" H 2800 8800 50  0001 C CNN
 	1    2800 8800
