File: Overview & Details/Audioboard/Audioboard_Activity/Audio_Board/Audio_Board.sch (KiCad schematic (older format))
At the start: 104 parts, among them J1 01x10 pinout, J1 1017523, J4 PBC03SAAN, J5 1017523, J6 1017521, J7 1017521, U1 VS1053B, U10 MOUNTINGHOLE2.5_THICK, U11 MOUNTINGHOLE2.5_THICK, U12 MOUNTINGHOLE2.5_THICK, U2 AP7312-1833W6-7, U3 MAX1735EUK25-T, U4 ADA4807-2, U5 ADA4807-2, U6 TC1262-2.5VDB, U7 MC78M12ABDTRKG, U8 TPA3250D2DDW-Amplifier_Audio, U9 MOUNTINGHOLE2.5_THICK, Y1 ABM8G-

Commit message: audio board error fixes
Parts:
- FB1, FB2: symbol Audio_Board-rescue:FERRITE_0603-Adafruit_VS1053_Breakout-eagle-import -> Audio_Board:FERRITE_0603-Adafruit_VS1053_Breakout-eagle-import
- U3: symbol Audio_Board-rescue:MAX1735EUK25+T-2019-02-05_05-23-06 -> Audio_Board:MAX1735EUK25+T-2019-02-05_05-23-06
- Y1: symbol Audio_Board-rescue:CRYSTAL3.2X2.5-Adafruit_VS1053_Breakout-eagle-import -> Audio_Board:CRYSTAL3.2X2.5-Adafruit_VS1053_Breakout-eagle-import
- renumbered J1 to J2
Connections:
- no-connect marks 28 -> 20
Changed lines of the file:
@@
 $EndComp
 $Comp
-L Audio_Board-rescue:CRYSTAL3.2X2.5-Adafruit_VS1053_Breakout-eagle-import Y1
+L Audio_Board:CRYSTAL3.2X2.5-Adafruit_VS1053_Breakout-eagle-import Y1
 U 1 1 5CCA6A9E
 P 1450 6100
@@
 $EndBitmap
 $Comp
-L Audio_Board-rescue:FERRITE_0603-Adafruit_VS1053_Breakout-eagle-import FB1
+L Audio_Board:FERRITE_0603-Adafruit_VS1053_Breakout-eagle-import FB1
 U 1 1 5C637F4B
 P 1550 2550
@@
 $EndComp
 $Comp
-L Audio_Board-rescue:FERRITE_0603-Adafruit_VS1053_Breakout-eagle-import FB2
+L Audio_Board:FERRITE_0603-Adafruit_VS1053_Breakout-eagle-import FB2
 U 1 1 5C68B93E
 P 2350 2350
@@
 0603
 $Comp
-L Audio_Board-rescue:MAX1735EUK25+T-2019-02-05_05-23-06 U3
+L Audio_Board:MAX1735EUK25+T-2019-02-05_05-23-06 U3
 U 1 1 5C7290D7
 P 6200 1900
@@
 NoConn ~ 2100 4100
 NoConn ~ 2100 4200
-NoConn ~ 2100 4800
 NoConn ~ 2100 4900
 NoConn ~ 2100 5000
 NoConn ~ 2100 5100
 NoConn ~ 2100 5200
-NoConn ~ 2100 5400
 NoConn ~ 2050 5600
 NoConn ~ 4900 5400
 NoConn ~ 4900 5600
 NoConn ~ 4900 5700
-NoConn ~ 4900 6000
-NoConn ~ 4900 6100
-NoConn ~ 4900 6200
-NoConn ~ 4900 6300
-NoConn ~ 4900 6400
 NoConn ~ 4900 6500
 Wire Wire Line
 	4650 4100 5000 4100
 NoConn ~ 5000 4100
-NoConn ~ 10350 3350
 $Comp
 L Audio_Board:TPA3250D2DDW-Amplifier_Audio U8
@@
 	5350 5500 4650 5500
 $Comp
-L Connector:Conn_01x10_Female J1
+L Connector:Conn_01x10_Female J2
 U 1 1 5FE2DB2F
 P 1950 8650
-F 0 "J1" H 1978 8626 50  0000 L CNN
+F 0 "J2" H 1978 8626 50  0000 L CNN
 F 1 "01x10 pinout" H 1978 8535 50  0000 L CNN
 F 2 "" H 1950 8650 50  0001 C CNN
@@
 $EndComp
 $Comp
-L power:GND #PWR?
+L power:GND #PWR0110
 U 1 1 5FE311AA
 P 1550 9150
-F 0 "#PWR?" H 1550 8900 50  0001 C CNN
+F 0 "#PWR0110" H 1550 8900 50  0001 C CNN
 F 1 "GND" H 1555 8977 50  0000 C CNN
 F 2 "" H 1550 9150 50  0001 C CNN
