File: Overview & Details/Audioboard/Audioboard_Activity/Audio_Board/Audio_Board.sch (KiCad schematic (older format))
At the start: 104 parts, among them J1 1017523, J2 01x10 pinout, J4 PBC03SAAN, J5 1017523, J6 1017521, J7 1017521, U1 VS1053B, U10 MOUNTINGHOLE2.5_THICK, U11 MOUNTINGHOLE2.5_THICK, U12 MOUNTINGHOLE2.5_THICK, U2 AP7312-1833W6-7, U3 MAX1735EUK25-T, U4 ADA4807-2, U5 ADA4807-2, U6 TC1262-2.5VDB, U7 MC78M12ABDTRKG, U8 TPA3250D2DDW-Amplifier_Audio, U9 MOUNTINGHOLE2.5_THICK, Y1 ABM8G-

Commit message: audio board lib file fixes
Parts:
- U10, U11, U12, U9: symbol Audio_Board-rescue:MOUNTINGHOLE2.5_THICK-Adafruit_VS1053_Breakout-eagle-import -> Audio_Board:MOUNTINGHOLE2.5_THICK-Adafruit_VS1053_Breakout-eagle-import
Connections:
- net labels added: Earth_w_GND-power
- net labels removed: Earth_w_GND, GND

Commit message: fixed footprint/symbol link for the MAX1735EUK25. created .pretty folder for AudioBoard footprints. the 1x10 pin connector for the sam32 still needs a footprint. the footprints for the phoenix conenctors are left uncompleted as an activity
Parts:
- U3: footprint 21-0057F -> Audio_Board:MAX1735EUK25&plus_T
Changed lines of the file:
@@
 EESchema Schematic File Version 4
-LIBS:Audio_Board-cache
 EELAYER 30 0
 EELAYER END
@@
 F 0 "U3" H 6925 2287 60  0000 C CNN
 F 1 "MAX1735EUK25-T" H 6925 2181 60  0000 C CNN
-F 2 "21-0057F" H 6925 2150 60  0001 C CNN
+F 2 "Audio_Board:MAX1735EUK25&plus_T" H 6925 2150 60  0001 C CNN
 F 3 "" H 6200 1900 60  0000 C CNN
 	1    6200 1900

Commit message: foottprintt instrtuctions
Parts:
- J2: footprint (none) -> Connector_PinHeader_2.54mm:PinHeader_1x10_P2.54mm_Vertical
- J5: footprint TerminalBlock_Phoenix:PhoenixContact_TermBlk_4P_SideEnt_6.35MM -> (none)
- J6: footprint TerminalBlock_Phoenix:PhoenixContact_TermBlk_2P_SideEnt_6.35MM -> (none); Description PCB Terminal Block, 4 Contact, TH -> PCB Terminal Block, 2 Contact, TH
- J7: footprint TerminalBlock_Phoenix:PhoenixContact_TermBlk_2P_SideEnt_6.35MM -> (none)
Changed lines of the file:
@@
 EESchema Schematic File Version 4
+LIBS:Audio_Board-cache
 EELAYER 30 0
 EELAYER END
@@
 F 0 "J6" H 15930 3042 50  0000 L CNN
 F 1 "1017521" H 15700 2850 50  0000 L CNN
-F 2 "TerminalBlock_Phoenix:PhoenixContact_TermBlk_2P_SideEnt_6.35MM" H 15850 3050 50  0001 C CNN
+F 2 "" H 15850 3050 50  0001 C CNN
 F 3 "https://www.phoenixcontact.com/online/portal/us/?uri=pxc-oc-itemdetail:pid=1017523&library=usen&pcck=P-11-01-05&tab=1&selectedCategory=ALL" H 15850 3050 50  0001 C CNN
-F 4 "PCB Terminal Block, 4 Contact, TH" H 15850 3050 50  0001 C CNN "Description"
+F 4 "PCB Terminal Block, 2 Contact, TH" H 15850 3050 50  0001 C CNN "Description"
 F 5 "" H 15850 3050 50  0001 C CNN "Package"
 F 6 "1017521" H 15850 3050 50  0001 C CNN "Part Number"
@@
 F 0 "J5" V 13514 912 50  0000 R CNN
 F 1 "1017523" V 13423 912 50  0000 R CNN
-F 2 "TerminalBlock_Phoenix:PhoenixContact_TermBlk_4P_SideEnt_6.35MM" H 13550 1200 50  0001 C CNN
+F 2 "" H 13550 1200 50  0001 C CNN
 F 3 "https://www.phoenixcontact.com/online/portal/us/?uri=pxc-oc-itemdetail:pid=1017523&library=usen&pcck=P-11-01-05&tab=1&selectedCategory=ALL" H 13550 1200 50  0001 C CNN
 F 4 "PCB Terminal Block, 4 Position, Through Hole, Push-in Spring connection" V 13550 1200 50  0001 C CNN "Description"
@@
 F 0 "J7" H 15930 5292 50  0000 L CNN
 F 1 "1017521" H 15700 5100 50  0000 L CNN
-F 2 "TerminalBlock_Phoenix:PhoenixContact_TermBlk_2P_SideEnt_6.35MM" H 15850 5300 50  0001 C CNN
+F 2 "" H 15850 5300 50  0001 C CNN
 F 3 "https://www.phoenixcontact.com/online/portal/us/?uri=pxc-oc-itemdetail:pid=1017523&library=usen&pcck=P-11-01-05&tab=1&selectedCategory=ALL" H 15850 5300 50  0001 C CNN
 F 4 "PCB Terminal Block, 4 Contact, TH" H 15850 5300 50  0001 C CNN "Description"
@@
 F 0 "J2" H 1978 8626 50  0000 L CNN
 F 1 "01x10 pinout" H 1978 8535 50  0000 L CNN
-F 2 "" H 1950 8650 50  0001 C CNN
+F 2 "Connector_PinHeader_2.54mm:PinHeader_1x10_P2.54mm_Vertical" H 1950 8650 50  0001 C CNN
 F 3 "~" H 1950 8650 50  0001 C CNN
 	1    1950 8650
