File: Overview & Details/LEDboard/LEDboard_Activity/LED_Board_s_.kicad_pcb (KiCad board)
At the start: 2 copper layers, 0 parts

Commit message: Removed erroneous ground plane
Routing:
- net GND: track 7.85 -> 0.00 mm
- removed copper zone on B.Cu, net GND
Changed lines of the file:
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@@
-(kicad_pcb (version 20171130) (host pcbnew "(5.1.5)-3")
+(kicad_pcb (version 20171130) (host pcbnew "(5.1.5-0-10_14)")
   (general
     (thickness 1.6)
     (drawings 0)
-    (tracks 7)
+    (tracks 0)
     (zones 0)
     (modules 0)
-    (nets 2)
+    (nets 1)
   )
   (page A4)
   (layers
     (0 F.Cu signal)
-    (31 B.Cu signal hide)
+    (31 B.Cu signal)
     (32 B.Adhes user)
     (33 F.Adhes user)
@@
   )
   (net 0 "")
-  (net 1 GND)
   (net_class Default "This is the default net class."
     (clearance 0.2)
@@
     (uvia_dia 0.3)
     (uvia_drill 0.1)
-    (add_net GND)
-  )
-  (segment (start 112.395 90.481685) (end 111.436685 91.44) (width 0.2) (layer B.Cu) (net 1))
-  (segment (start 112.395 89.916) (end 112.395 90.481685) (width 0.2) (layer B.Cu) (net 1))
-  (segment (start 111.436685 91.44) (end 111.436685 93.160315) (width 0.2) (layer B.Cu) (net 1))
-  (segment (start 111.436685 93.160315) (end 110.744 93.853) (width 0.2) (layer B.Cu) (net 1))
-  (segment (start 147.047001 90.315999) (end 146.539001 90.315999) (width 0.2) (layer B.Cu) (net 1))
-  (segment (start 147.447 89.916) (end 147.047001 90.315999) (width 0.2) (layer B.Cu) (net 1))
-  (segment (start 95.123 108.966) (end 93.599 110.49) (width 0.2) (layer B.Cu) (net 1))
-  (zone (net 1) (net_name GND) (layer B.Cu) (hatch full 0.508)
-    (connect_pads (clearance 0.508))
-    (min_thickness 0.254)
-    (fill yes (arc_segments 32) (thermal_gap 0.508) (thermal_bridge_width 0.508))
-    (polygon
-      (pts
-        (xy 193.04 133.096) (xy 80.137 132.969) (xy 80.137 62.611) (xy 80.2005 62.611) (xy 80.264 62.611)
-        (xy 80.137 58.293) (xy 193.04 58.293)
-      )
-    )
-  )
-  (zone (net 1) (net_name GND) (layer B.Cu) (hatch full 0.508)
-    (connect_pads (clearance 0.508))
-    (min_thickness 0.254)
-    (fill yes (arc_segments 32) (thermal_gap 0.508) (thermal_bridge_width 0.508))
-    (polygon
-      (pts
-        (xy 191.643 117.475) (xy 183.896 117.475) (xy 183.769 73.66) (xy 191.643 73.66)
-      )
-    )
-  )
-  (zone (net 1) (net_name GND) (layer B.Cu) (hatch full 0.508)
-    (connect_pads (clearance 0.508))
-    (min_thickness 0.254)
-    (fill yes (arc_segments 32) (thermal_gap 0.508) (thermal_bridge_width 0.508))
-    (polygon
-      (pts
-        (xy 191.262 117.475) (xy 183.769 117.475) (xy 183.769 73.66) (xy 191.262 73.66)
-      )
-    )
   )
 )
