File: Overview & Details/Powerboard/Powerboard_Activity/Power_Board.sch (KiCad schematic (older format))
At the start: 43 parts

Commit message: removed portion for acitivty and fixed libraries
Parts:
- removed C?: 47µF @ 10V, symbol Device:CP1
- removed C?: 1µF, symbol Device:C
- removed C?: 100µF, symbol Device:CP1
- removed C?: 82pF, symbol Device:C
- removed C?: 10µF, symbol Device:CP1
- removed C?: 22µF @ 10V, symbol Device:CP1
- removed D?: PMEG2010AEH, symbol Device:D_Schottky
- removed L?: 10µH, symbol Device:L
- removed L?: 22µH, symbol Device:L
- removed R?: 130kΩ, symbol Device:R_Small_US
- removed R?: 300kΩ, symbol Device:R_Small_US
- removed U?: MAX735CSA, symbol Regulator_Switching:MAX735CSA
Connections:
- wire segments 122 -> 93

Commit message: activity finalizing
Parts:
- removed J? (x2): Conn_01x02, symbol Connector_Generic:Conn_01x02
Changed lines of the file:
@@
 @ 16V
-$Comp
-L Connector_Generic:Conn_01x02 J?
-U 1 1 5EC5DED5
-P 2600 9100
-F 0 "J?" H 2680 9092 50  0000 L CNN
-F 1 "Conn_01x02" H 2680 9001 50  0000 L CNN
-F 2 "" H 2600 9100 50  0001 C CNN
-F 3 "~" H 2600 9100 50  0001 C CNN
-	1    2600 9100
-	1    0    0    -1
-$EndComp
-$Comp
-L Connector_Generic:Conn_01x02 J?
-U 1 1 5EC5F668
-P 4150 9050
-F 0 "J?" H 4230 9042 50  0000 L CNN
-F 1 "Conn_01x02" H 4230 8951 50  0000 L CNN
-F 2 "" H 4150 9050 50  0001 C CNN
-F 3 "~" H 4150 9050 50  0001 C CNN
-	1    4150 9050
-	1    0    0    -1
-$EndComp
 $Comp
 L power:PWR_FLAG #FLG0101
