File: Overview & Details/Powerboard/Powerboard_Activity/Power_Board.sch (KiCad schematic (older format))
At the start: 29 parts

Commit message: added diode footprint
Parts:
- D? (x4): footprint Package_TO_SOT_SMD:TO-252AA_TabPin4 -> (none)
Changed lines of the file:
@@
 EESchema Schematic File Version 4
+LIBS:Power_Board-cache
 EELAYER 30 0
 EELAYER END
@@
 F 0 "D?" V 12604 3179 50  0000 L CNN
 F 1 "VS-MURD620CT-M3" V 12800 3150 50  0000 L CNN
-F 2 "Package_TO_SOT_SMD:TO-252AA_TabPin4" H 12650 3100 50  0001 C CNN
+F 2 "" H 12650 3100 50  0001 C CNN
 F 3 "https://www.vishay.com/docs/93497/vs-murd620c.pdf" H 12650 3100 50  0001 C CNN
 	1    12650 3100
@@
 F 0 "D?" V 6604 3179 50  0000 L CNN
 F 1 "VS-MURD620CT-M3" V 6800 3150 50  0000 L CNN
-F 2 "Package_TO_SOT_SMD:TO-252AA_TabPin4" H 6650 3100 50  0001 C CNN
+F 2 "" H 6650 3100 50  0001 C CNN
 F 3 "https://www.vishay.com/docs/93497/vs-murd620c.pdf" H 6650 3100 50  0001 C CNN
 	1    6650 3100
@@
 F 0 "D?" V 3904 6529 50  0000 L CNN
 F 1 "VS-MURD620CT-M3" V 4100 6500 50  0000 L CNN
-F 2 "Package_TO_SOT_SMD:TO-252AA_TabPin4" H 3950 6450 50  0001 C CNN
+F 2 "" H 3950 6450 50  0001 C CNN
 F 3 "https://www.vishay.com/docs/93497/vs-murd620c.pdf" H 3950 6450 50  0001 C CNN
 	1    3950 6450
@@
 F 0 "D?" V 8104 6429 50  0000 L CNN
 F 1 "VS-MURD620CT-M3" V 8300 6400 50  0000 L CNN
-F 2 "Package_TO_SOT_SMD:TO-252AA_TabPin4" H 8150 6350 50  0001 C CNN
+F 2 "" H 8150 6350 50  0001 C CNN
 F 3 "https://www.vishay.com/docs/93497/vs-murd620c.pdf" H 8150 6350 50  0001 C CNN
 	1    8150 6350
@@
 	11900 9700 11900 9950
 $Comp
-L Power_Board:+5VR #PWR?
+L Power_Board:+5VR #PWR0129
 U 1 1 5EACA33B
 P 13400 1900
-F 0 "#PWR?" H 13400 1750 50  0001 C CNN
+F 0 "#PWR0129" H 13400 1750 50  0001 C CNN
 F 1 "+5VR" H 13415 2073 50  0000 C CNN
 F 2 "" H 13400 1900 50  0001 C CNN
@@
 	10675 4850 10675 7025
 $Comp
-L Power_Board:+5VR #PWR?
+L Power_Board:+5VR #PWR0131
 U 1 1 5EAF8C5D
 P 11400 9700
-F 0 "#PWR?" H 11400 9550 50  0001 C CNN
+F 0 "#PWR0131" H 11400 9550 50  0001 C CNN
 F 1 "+5VR" H 11415 9873 50  0000 C CNN
 F 2 "" H 11400 9700 50  0001 C CNN
