File: Overview & Details/Displayboard/Displayboard_Activity/Display_Board/Display_Board.sch (KiCad schematic (older format))
At the start: 0 parts

Commit message: created connector
Parts:
- added J?: Conn_01x50, symbol Display_Board:Conn_01x50
Changed lines of the file:
@@
 EESchema Schematic File Version 4
+LIBS:Display_Board-cache
 EELAYER 30 0
 EELAYER END
@@
 Text Notes 4150 5625 0    118  ~ 24
 Display TFT
+$Comp
+L Display_Board:Conn_01x50 J?
+U 1 1 5EC95D65
+P 10050 3825
+F 0 "J?" H 10022 3751 50  0000 R CNN
+F 1 "Conn_01x50" H 10022 3842 50  0000 R CNN
+F 2 "" H 10000 1075 50  0001 C CNN
+F 3 "" H 10000 1075 50  0001 C CNN
+	1    10050 3825
+	-1   0    0    1
+$EndComp
 $EndSCHEMATC

Commit message: labels added. Go ham
Connections:
- net LEDK: now reaches J?.1
- net LCD_RST: now reaches J?.10
- net VSYNC: now reaches J?.11
- net HSYNC: now reaches J?.12
- net DOTCLK: now reaches J?.13
- net DE: now reaches J?.14
- net DB17: now reaches J?.15
- net DB16: now reaches J?.16
- net DB15: now reaches J?.17
- net DB14: now reaches J?.18
- net DB13: now reaches J?.19
- net LEDA1: now reaches J?.2
- net DB12: now reaches J?.20
- net DB11: now reaches J?.21
- net DB10: now reaches J?.22
- net DB09: now reaches J?.23
- net DB08: now reaches J?.24
- net LCD_DATA7: now reaches J?.25
- net LCD_DATA6: now reaches J?.26
- net LCD_DATA5: now reaches J?.27
- net LCD_DATA4: now reaches J?.28
- net LCD_DATA3: now reaches J?.29
- net LEDA2: now reaches J?.3
- net LCD_DATA2: now reaches J?.30
- net LCD_DATA1: now reaches J?.31
- net LCD_DATA0: now reaches J?.32
- net SDO: now reaches J?.33
- net SDI_3V: now reaches J?.34
- net LCD_RD: now reaches J?.35
- net LCD_WR: now reaches J?.36
- net LCD_RS: now reaches J?.37
- net LCD_CS: now reaches J?.38
- net TE: now reaches J?.39
- net LEDA3: now reaches J?.4
- net Vdd_40: now reaches J?.40
- net Vdd_41: now reaches J?.41
- net Vel_42: now reaches J?.42
- net GND_43: now reaches J?.43
- net LCD_X+: now reaches J?.44
- net LCD_Y+: now reaches J?.45
- net LCD_X-: now reaches J?.46
- net LCD_Y-: now reaches J?.47
- net GND_48: now reaches J?.48
- net GND_49: now reaches J?.49
- net LEDA4: now reaches J?.5
- net GND_50: now reaches J?.50
- net IM0: now reaches J?.6
- net IM1: now reaches J?.7
- net IM2: now reaches J?.8
- net IM3: now reaches J?.9
Changed lines of the file:
@@
 	-1   0    0    1
 $EndComp
+Text Label 9850 1325 2    50   ~ 0
+GND_50
+Text Label 9850 1425 2    50   ~ 0
+GND_49
+Text Label 9850 1525 2    50   ~ 0
+GND_48
+Text Label 9850 1625 2    50   ~ 0
+LCD_Y-
+Text Label 9850 1725 2    50   ~ 0
+LCD_X-
+Text Label 9850 1825 2    50   ~ 0
+LCD_Y+
+Text Label 9850 1925 2    50   ~ 0
+LCD_X+
+Text Label 9850 2025 2    50   ~ 0
+GND_43
+Text Label 9850 2125 2    50   ~ 0
+Vel_42
+Text Label 9850 2225 2    50   ~ 0
+Vdd_41
+Text Label 9850 2325 2    50   ~ 0
+Vdd_40
+Text Label 9850 2425 2    50   ~ 0
+TE
+Text Label 9850 2525 2    50   ~ 0
+LCD_CS
+Text Label 9850 2625 2    50   ~ 0
+LCD_RS
+Text Label 9850 2725 2    50   ~ 0
+LCD_WR
+Text Label 9850 2825 2    50   ~ 0
+LCD_RD
+Text Label 9850 2925 2    50   ~ 0
+SDI_3V
+Text Label 9850 3025 2    50   ~ 0
+SDO
+Text Label 9850 3125 2    50   ~ 0
+LCD_DATA0
+Text Label 9850 3225 2    50   ~ 0
+LCD_DATA1
+Text Label 9850 3325 2    50   ~ 0
+LCD_DATA2
+Text Label 9850 3425 2    50   ~ 0
+LCD_DATA3
+Text Label 9850 3525 2    50   ~ 0
+LCD_DATA4
+Text Label 9850 3625 2    50   ~ 0
+LCD_DATA5
+Text Label 9850 3725 2    50   ~ 0
+LCD_DATA6
+Text Label 9850 3825 2    50   ~ 0
+LCD_DATA7
+Text Label 9850 3925 2    50   ~ 0
+DB08
+Text Label 9850 4025 2    50   ~ 0
+DB09
+Text Label 9850 4125 2    50   ~ 0
+DB10
+Text Label 9850 4225 2    50   ~ 0
+DB11
+Text Label 9850 4325 2    50   ~ 0
+DB12
+Text Label 9850 4425 2    50   ~ 0
+DB13
+Text Label 9850 4525 2    50   ~ 0
+DB14
+Text Label 9850 4625 2    50   ~ 0
+DB15
+Text Label 9850 4725 2    50   ~ 0
+DB16
+Text Label 9850 4825 2    50   ~ 0
+DB17
+Text Label 9850 4925 2    50   ~ 0
+DE
+Text Label 9850 5025 2    50   ~ 0
+DOTCLK
+Text Label 9850 5125 2    50   ~ 0
+HSYNC
+Text Label 9850 5225 2    50   ~ 0
+VSYNC
+Text Label 9850 5325 2    50   ~ 0
+LCD_RST
+Text Label 9850 5425 2    50   ~ 0
+IM3
+Text Label 9850 5525 2    50   ~ 0
+IM2
+Text Label 9850 5625 2    50   ~ 0
+IM1
+Text Label 9850 5725 2    50   ~ 0
+IM0
+Text Label 9850 5825 2    50   ~ 0
+LEDA4
+Text Label 9850 5925 2    50   ~ 0
+LEDA3
+Text Label 9850 6025 2    50   ~ 0
+LEDA2
+Text Label 9850 6125 2    50   ~ 0
+LEDA1
+Text Label 9850 6225 2    50   ~ 0
+LEDK
 $EndSCHEMATC
