File: Overview & Details/Displayboard/Displayboard_Activity/Display_Board/Root.sch (KiCad schematic (older format))
At the start: 37 parts, among them J1 Micro_SD_Card_Det_MOD-Connect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, J2 Conn_01x20_Female, J4 Conn_01x20_Female, Q1 MMBT2222A-TP-dk_Transistors-B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, U1 MCP130T-300I_TT-dk_PMIC-Super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, U2 SN74LVC245AN-dk_Logic-Buffers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, U3 STMPE811QTR-Interface_Expansi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, U4 SN74LVC245AN-dk_Logic-Buffers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, U5 LP2988-3.3_SOIC8_VSSOP8

Commit message: Use hand_solder footprints
Parts:
- C1, C2, C3, C4, C5, C6, C7, C8, C9: footprint Capacitor_SMD:C_0805_2012Metric -> Capacitor_SMD:C_0805_2012Metric_Pad1.15x1.40mm_HandSolder
- R1, R10, R11, R12, R13, R14, R15, R2, R3, R4, R5, R6, R7, R8, R9: footprint Resistor_SMD:R_0805_2012Metric -> Resistor_SMD:R_0805_2012Metric_Pad1.15x1.40mm_HandSolder
Changed lines of the file:
@@
 F 0 "R11" H 9753 2906 50  0000 L CNN
 F 1 "10Ω" H 9753 2815 50  0000 L CNN
-F 2 "Resistor_SMD:R_0805_2012Metric" H 9685 2860 50  0001 C CNN
+F 2 "Resistor_SMD:R_0805_2012Metric_Pad1.15x1.40mm_HandSolder" H 9685 2860 50  0001 C CNN
 F 3 "~" H 9685 2860 50  0001 C CNN
 	1    9685 2860
@@
 F 0 "R10" H 9453 2906 50  0000 L CNN
 F 1 "10Ω" H 9453 2815 50  0000 L CNN
-F 2 "Resistor_SMD:R_0805_2012Metric" H 9385 2860 50  0001 C CNN
+F 2 "Resistor_SMD:R_0805_2012Metric_Pad1.15x1.40mm_HandSolder" H 9385 2860 50  0001 C CNN
 F 3 "~" H 9385 2860 50  0001 C CNN
 	1    9385 2860
@@
 F 0 "R9" H 9153 2906 50  0000 L CNN
 F 1 "10Ω" H 9153 2815 50  0000 L CNN
-F 2 "Resistor_SMD:R_0805_2012Metric" H 9085 2860 50  0001 C CNN
+F 2 "Resistor_SMD:R_0805_2012Metric_Pad1.15x1.40mm_HandSolder" H 9085 2860 50  0001 C CNN
 F 3 "~" H 9085 2860 50  0001 C CNN
 	1    9085 2860
@@
 F 0 "R8" H 8853 2906 50  0000 L CNN
 F 1 "10Ω" H 8853 2815 50  0000 L CNN
-F 2 "Resistor_SMD:R_0805_2012Metric" H 8785 2860 50  0001 C CNN
+F 2 "Resistor_SMD:R_0805_2012Metric_Pad1.15x1.40mm_HandSolder" H 8785 2860 50  0001 C CNN
 F 3 "~" H 8785 2860 50  0001 C CNN
 	1    8785 2860
@@
 F 0 "R3" V 9110 2140 50  0000 C CNN
 F 1 "1kΩ" V 9310 2140 50  0000 C CNN
-F 2 "Resistor_SMD:R_0805_2012Metric" H 9200 2145 50  0001 C CNN
+F 2 "Resistor_SMD:R_0805_2012Metric_Pad1.15x1.40mm_HandSolder" H 9200 2145 50  0001 C CNN
 F 3 "~" H 9200 2145 50  0001 C CNN
 	1    9200 2145
@@
 F 0 "C1" H 5497 6966 50  0000 L CNN
 F 1 "0.1µF" H 5497 6875 50  0000 L CNN
-F 2 "Capacitor_SMD:C_0805_2012Metric" H 5405 6920 50  0001 C CNN
+F 2 "Capacitor_SMD:C_0805_2012Metric_Pad1.15x1.40mm_HandSolder" H 5405 6920 50  0001 C CNN
 F 3 "~" H 5405 6920 50  0001 C CNN
 	1    5405 6920
@@
 F 0 "R13" H 5943 6981 50  0000 L CNN
 F 1 "10kΩ" H 5943 6890 50  0000 L CNN
-F 2 "Resistor_SMD:R_0805_2012Metric" H 5875 6935 50  0001 C CNN
+F 2 "Resistor_SMD:R_0805_2012Metric_Pad1.15x1.40mm_HandSolder" H 5875 6935 50  0001 C CNN
 F 3 "~" H 5875 6935 50  0001 C CNN
 	1    5875 6935
@@
 F 0 "C8" H 4682 9511 50  0000 L CNN
 F 1 "0.1µF" H 4682 9420 50  0000 L CNN
-F 2 "Capacitor_SMD:C_0805_2012Metric" H 4590 9465 50  0001 C CNN
+F 2 "Capacitor_SMD:C_0805_2012Metric_Pad1.15x1.40mm_HandSolder" H 4590 9465 50  0001 C CNN
 F 3 "~" H 4590 9465 50  0001 C CNN
 	1    4590 9465
@@
 F 0 "C7" H 6776 9226 50  0000 L CNN
 F 1 "4.7µF" H 6776 9135 50  0000 L CNN
-F 2 "Capacitor_SMD:C_0805_2012Metric" H 6685 9180 50  0001 C CNN
+F 2 "Capacitor_SMD:C_0805_2012Metric_Pad1.15x1.40mm_HandSolder" H 6685 9180 50  0001 C CNN
 F 3 "~" H 6685 9180 50  0001 C CNN
 	1    6685 9180
@@
 F 0 "C6" H 6397 9226 50  0000 L CNN
 F 1 "0.1µF" H 6397 9135 50  0000 L CNN
-F 2 "Capacitor_SMD:C_0805_2012Metric" H 6305 9180 50  0001 C CNN
+F 2 "Capacitor_SMD:C_0805_2012Metric_Pad1.15x1.40mm_HandSolder" H 6305 9180 50  0001 C CNN
 F 3 "~" H 6305 9180 50  0001 C CNN
 	1    6305 9180
@@
 F 0 "C9" H 5842 9526 50  0000 L CNN
 F 1 "0.01µF" H 5842 9435 50  0000 L CNN
-F 2 "Capacitor_SMD:C_0805_2012Metric" H 5750 9480 50  0001 C CNN
+F 2 "Capacitor_SMD:C_0805_2012Metric_Pad1.15x1.40mm_HandSolder" H 5750 9480 50  0001 C CNN
 F 3 "~" H 5750 9480 50  0001 C CNN
 	1    5750 9480
@@
 F 0 "R15" H 5973 9226 50  0000 L CNN
 F 1 "330kΩ" H 5973 9135 50  0000 L CNN
-F 2 "Resistor_SMD:R_0805_2012Metric" H 5905 9180 50  0001 C CNN
+F 2 "Resistor_SMD:R_0805_2012Metric_Pad1.15x1.40mm_HandSolder" H 5905 9180 50  0001 C CNN
 F 3 "~" H 5905 9180 50  0001 C CNN
 	1    5905 9180
@@
 F 0 "C3" H 9706 6996 50  0000 L CNN
 F 1 "10µF" H 9706 6905 50  0000 L CNN
-F 2 "Capacitor_SMD:C_0805_2012Metric" H 9615 6950 50  0001 C CNN
+F 2 "Capacitor_SMD:C_0805_2012Metric_Pad1.15x1.40mm_HandSolder" H 9615 6950 50  0001 C CNN
 F 3 "~" H 9615 6950 50  0001 C CNN
 	1    9615 6950
@@
 F 0 "C2" H 9327 6996 50  0000 L CNN
 F 1 "0.1µF" H 9327 6905 50  0000 L CNN
-F 2 "Capacitor_SMD:C_0805_2012Metric" H 9235 6950 50  0001 C CNN
+F 2 "Capacitor_SMD:C_0805_2012Metric_Pad1.15x1.40mm_HandSolder" H 9235 6950 50  0001 C CNN
 F 3 "~" H 9235 6950 50  0001 C CNN
 	1    9235 6950
@@
 F 0 "C5" H 4091 9226 50  0000 L CNN
 F 1 "10µF" H 4091 9135 50  0000 L CNN
-F 2 "Capacitor_SMD:C_0805_2012Metric" H 4000 9180 50  0001 C CNN
+F 2 "Capacitor_SMD:C_0805_2012Metric_Pad1.15x1.40mm_HandSolder" H 4000 9180 50  0001 C CNN
 F 3 "~" H 4000 9180 50  0001 C CNN
 	1    4000 9180
@@
 F 0 "C4" H 3712 9226 50  0000 L CNN
 F 1 "0.1µF" H 3712 9135 50  0000 L CNN
-F 2 "Capacitor_SMD:C_0805_2012Metric" H 3620 9180 50  0001 C CNN
+F 2 "Capacitor_SMD:C_0805_2012Metric_Pad1.15x1.40mm_HandSolder" H 3620 9180 50  0001 C CNN
 F 3 "~" H 3620 9180 50  0001 C CNN
 	1    3620 9180
@@
 F 0 "R2" H 8858 1806 50  0000 L CNN
 F 1 "10Ω" H 8858 1715 50  0000 L CNN
-F 2 "Resistor_SMD:R_0805_2012Metric" H 8790 1760 50  0001 C CNN
+F 2 "Resistor_SMD:R_0805_2012Metric_Pad1.15x1.40mm_HandSolder" H 8790 1760 50  0001 C CNN
 F 3 "~" H 8790 1760 50  0001 C CNN
 	1    8790 1760
@@
 F 0 "R1" H 4913 1781 50  0000 L CNN
 F 1 "10kΩ" H 4913 1690 50  0000 L CNN
-F 2 "Resistor_SMD:R_0805_2012Metric" H 4845 1735 50  0001 C CNN
+F 2 "Resistor_SMD:R_0805_2012Metric_Pad1.15x1.40mm_HandSolder" H 4845 1735 50  0001 C CNN
 F 3 "~" H 4845 1735 50  0001 C CNN
 	1    4845 1735
@@
 F 0 "R12" H 7288 5631 50  0000 L CNN
 F 1 "10kΩ" H 7288 5540 50  0000 L CNN
-F 2 "Resistor_SMD:R_0805_2012Metric" H 7220 5585 50  0001 C CNN
+F 2 "Resistor_SMD:R_0805_2012Metric_Pad1.15x1.40mm_HandSolder" H 7220 5585 50  0001 C CNN
 F 3 "~" H 7220 5585 50  0001 C CNN
 	1    7220 5585
@@
 F 0 "R7" H 3633 2536 50  0000 L CNN
 F 1 "10kΩ" H 3633 2445 50  0000 L CNN
-F 2 "Resistor_SMD:R_0805_2012Metric" H 3565 2490 50  0001 C CNN
+F 2 "Resistor_SMD:R_0805_2012Metric_Pad1.15x1.40mm_HandSolder" H 3565 2490 50  0001 C CNN
 F 3 "~" H 3565 2490 50  0001 C CNN
 	1    3565 2490
@@
 F 0 "R6" H 3333 2536 50  0000 L CNN
 F 1 "10kΩ" H 3333 2445 50  0000 L CNN
-F 2 "Resistor_SMD:R_0805_2012Metric" H 3265 2490 50  0001 C CNN
+F 2 "Resistor_SMD:R_0805_2012Metric_Pad1.15x1.40mm_HandSolder" H 3265 2490 50  0001 C CNN
 F 3 "~" H 3265 2490 50  0001 C CNN
 	1    3265 2490
@@
 F 0 "R5" H 3033 2536 50  0000 L CNN
 F 1 "10kΩ" H 3033 2445 50  0000 L CNN
-F 2 "Resistor_SMD:R_0805_2012Metric" H 2965 2490 50  0001 C CNN
+F 2 "Resistor_SMD:R_0805_2012Metric_Pad1.15x1.40mm_HandSolder" H 2965 2490 50  0001 C CNN
 F 3 "~" H 2965 2490 50  0001 C CNN
 	1    2965 2490
@@
 F 0 "R4" H 2733 2536 50  0000 L CNN
 F 1 "10kΩ" H 2733 2445 50  0000 L CNN
-F 2 "Resistor_SMD:R_0805_2012Metric" H 2665 2490 50  0001 C CNN
+F 2 "Resistor_SMD:R_0805_2012Metric_Pad1.15x1.40mm_HandSolder" H 2665 2490 50  0001 C CNN
 F 3 "~" H 2665 2490 50  0001 C CNN
 	1    2665 2490
@@
 F 0 "R14" H 9088 7861 50  0000 L CNN
 F 1 "10kΩ" H 9088 7770 50  0000 L CNN
-F 2 "Resistor_SMD:R_0805_2012Metric" H 9020 7815 50  0001 C CNN
+F 2 "Resistor_SMD:R_0805_2012Metric_Pad1.15x1.40mm_HandSolder" H 9020 7815 50  0001 C CNN
 F 3 "~" H 9020 7815 50  0001 C CNN
 	1    9020 7815

Commit message: I forgot to save...
Parts:
- J1: footprint Connector_Card:microSD_HC_Molex_104031-0811 -> Display_Board:503182-1852
Changed lines of the file:
@@
 F 0 "J1" H 7220 1926 50  0000 L CNN
 F 1 "Micro_SD_Card_Det_MOD-Connector" H 7220 1835 50  0000 L CNN
-F 2 "Connector_Card:microSD_HC_Molex_104031-0811" H 8440 2580 50  0001 C CNN
+F 2 "Display_Board:503182-1852" H 8440 2580 50  0001 C CNN
 F 3 "" H 6390 1980 50  0001 C CNN
 	1    6390 1880

Commit message: Add new symbols to library with a different name
Parts:
- J1: symbol Display_Board:Micro_SD_Card_Det_MOD-Connector -> Display_Board_2:Micro_SD_Card_Det_MOD-Connector
- Q1: symbol Display_Board:MMBT2222A-TP-dk_Transistors-Bipolar-BJT-Single -> Display_Board_2:MMBT2222A-TP-dk_Transistors-Bipolar-BJT-Single
- U1: symbol Display_Board:MCP130T-300I_TT-dk_PMIC-Supervisors -> Display_Board_2:MCP130T-300I_TT-dk_PMIC-Supervisors
- U2, U4: symbol Display_Board:SN74LVC245AN-dk_Logic-Buffers-Drivers-Receivers-Transceivers -> Display_Board_2:SN74LVC245AN-dk_Logic-Buffers-Drivers-Receivers-Transceivers
- U3: symbol Display_Board:STMPE811QTR-Interface_Expansion -> Display_Board_2:STMPE811QTR-Interface_Expansion
Changed lines of the file:
@@
 NoConn ~ 5490 1730
 $Comp
-L Display_Board:Micro_SD_Card_Det_MOD-Connector J1
+L Display_Board_2:Micro_SD_Card_Det_MOD-Connector J1
 U 1 1 5ECFB234
 P 6390 1880
@@
 	4845 1930 5490 1930
 $Comp
-L Display_Board:SN74LVC245AN-dk_Logic-Buffers-Drivers-Receivers-Transceivers U2
+L Display_Board_2:SN74LVC245AN-dk_Logic-Buffers-Drivers-Receivers-Transceivers U2
 U 1 1 5EDC62A5
 P 5540 4725
@@
 $EndComp
 $Comp
-L Display_Board:SN74LVC245AN-dk_Logic-Buffers-Drivers-Receivers-Transceivers U4
+L Display_Board_2:SN74LVC245AN-dk_Logic-Buffers-Drivers-Receivers-Transceivers U4
 U 1 1 5EDC87AA
 P 8175 4685
@@
 $EndComp
 $Comp
-L Display_Board:MCP130T-300I_TT-dk_PMIC-Supervisors U1
+L Display_Board_2:MCP130T-300I_TT-dk_PMIC-Supervisors U1
 U 1 1 5EDCBEFA
 P 5020 7310
@@
 $EndComp
 $Comp
-L Display_Board:STMPE811QTR-Interface_Expansion U3
+L Display_Board_2:STMPE811QTR-Interface_Expansion U3
 U 1 1 5EDCD46F
 P 7635 7735
@@
 $EndComp
 $Comp
-L Display_Board:MMBT2222A-TP-dk_Transistors-Bipolar-BJT-Single Q1
+L Display_Board_2:MMBT2222A-TP-dk_Transistors-Bipolar-BJT-Single Q1
 U 1 1 5EDCF54B
 P 9600 2145
